File: Hardware/PIC_WeatherMonitor/PIC_WeatherMonitor.kicad_sch (KiCad schematic)
At the start: 0 parts

Commit message: v1.0 in progress
Parts:
- added C1, C3: 10uF, symbol Device:C
- added C2, C4: 0.1uF, symbol Device:C
- added C5, C6, C7: 100nF, symbol Device:C
- added J1: Barrel_Jack_Switch, symbol Connector:Barrel_Jack_Switch
- added R1: 1M, symbol Device:R
- added U1: ATWINC1500-MR210PB1961, ATWINC15x0-MR210_MCH, symbol ATWINC1500:ATWINC1500-MR210PB1961
- added U2: PIC16F18877-I/PT, TQFP44_PT_MCH, symbol PIC16:PIC16F18877-I_PT
- added U3: LD1117S33TR_SOT223, Package_TO_SOT_SMD:SOT-223-3_TabPin2, symbol Regulator_Linear:LD1117S12TR_SOT223
Connections:
- new net: C1.1, C2.1, J1.1, U3.3 (VI)
- new net: C6.2, U1.24 (1P3V_TP)
- new net: R1.2, U1.10 (SPI_CFG)
- new net +3.3V: C3.1, C4.1, U3.2 (VO)
- new net GND: C1.2, C2.2, C3.2, C4.2, C5.2, C6.1, C7.1, J1.2, J1.3, U1.12 (GND_2), U1.28 (GND_3), U1.29 (GND_PADDLE), U1.9 (GND_1), U3.1 (GND)
- new net VDD: C5.1, C7.2, R1.1, U1.20 (VBAT), U1.23 (VDDIO)
- new net WINC_CHIP_EN: U1.22 (CHIP_EN), U2.36 (RC2)
- new net WINC_EXTINT: U1.13 (IRQN), U2.1 (RC7)
- new net WINC_MISO: U1.17 (SPI_MISO), U2.42 (RC4)
- new net WINC_MOSI: U1.15 (SPI_MOSI), U2.43 (RC5)
- new net WINC_RESET: U2.44 (RC6)
- new net WINC_SCK: U1.18 (SPI_SCK), U2.37 (RC3)
- new net WINC_SS: U1.16 (SPI_SSN), U2.24 (RA5)
- new net WINC_WAKE: U1.11 (WAKE), U2.35 (RC1)
- no-connect marks 0 -> 34
